File: PCB_LTF1/LTF1.brd (EAGLE design)
At the start: 54 x 61 mm, 29 parts, among them Q1 BD139, Q4 BD139

Commit message: design rule passed
Parts:
- OPAMPKANAN: device linear:DIL08 -> op-amp-long:DIL08
- Q1, Q4: device transistor-power:TO126AV -> transistor-power-small-pad:TO126AV
- moved R11 2.00 mm to (28.1, 18.8)
- moved R4 2.00 mm to (24.3, 18.8)
- moved R7 2.00 mm to (31.9, 18.8)
- moved R8 2.00 mm to (35.7, 18.8)
- moved Q1 1.41 mm to (17.7, 19.8)
- moved IRL 1.00 mm to (23.0, 51.6)
- moved MOTORDRIVER 1.00 mm to (8.92, 18.4)
- moved R12 1.00 mm to (15.4, 9.13)
- moved R2 1.00 mm to (31.6, 42.4)
- moved R6 1.00 mm to (35.8, 42.7)
- moved R9 1.00 mm to (9.04, 24.4)
Routing:
- net +5V: track 157.9 -> 162.1 mm
- net N$3: track 18.5 -> 20.7 mm
- net N$5: track 15.4 -> 13.4 mm
- net 0: track 242.6 -> 244.6 mm
- net N$4: track 23.5 -> 24.9 mm
- net N$6: track 27.9 -> 29.1 mm
- net N$1: track 7.44 -> 6.44 mm
- net N$8: track 16.5 -> 15.5 mm
- net MOTORKANAN1: track 14.4 -> 15.3 mm
- net N$10: track 22.4 -> 21.7 mm
- net N$7: track 17.3 -> 17.9 mm
- net IRKIRI: track 13.5 -> 12.9 mm
