File: PCB_LTF1/LTF1.sch (EAGLE design)
At the start: 29 parts, among them Q1 BD139, Q4 BD139

Commit message: design rule passed
Parts:
- OPAMPKANAN: device linear:LM358N -> op-amp-long:LM358N
- Q1, Q4: device transistor-power:BD139 -> transistor-power-small-pad:BD139
